File: t1.kicad_pcb (KiCad board)
At the start: 4 copper layers, 63 x 35.6 mm, 47 parts, among them J1 Barrel_Jack_Switch, J2 USB_B, J3 P1, J4 2x2M, J5 ICSP1, J6 P2, U1 ATmega8U2-AU, Y1 16MHz

Commit message: Test
Parts:
- removed H1, H4: MountingHole, MountingHole:MountingHole_2.7mm_M2.5
